Commit message: Actualizacion de archivos launch

File: ulite6_arm_description/urdf/mech/ulite6_arm.urdf.xacro (robot description, xacro)
@@ -17,8 +17,8 @@
     <xacro:property name="default_inertial_params_filename" value="xarm6_type9_HT_BR2"/>
     <xacro:if value="${inertial_params_filename != ''}">
-      <xacro:property name="link_inertial_params_file" value="$(find xarm_description)/config/link_inertial/${inertial_params_filename}.yaml"/>
+      <xacro:property name="link_inertial_params_file" value="$(find ulite6_arm_description)/config/link_inertial/${inertial_params_filename}.yaml"/>
     </xacro:if>
     <xacro:unless value="${inertial_params_filename != ''}">
-      <xacro:property name="link_inertial_params_file" value="$(find xarm_description)/config/link_inertial/${default_inertial_params_filename}.yaml"/>
+      <xacro:property name="link_inertial_params_file" value="$(find ulite6_arm_description)/config/link_inertial/${default_inertial_params_filename}.yaml"/>
     </xacro:unless>
     <xacro:if value="${use_xacro_load_yaml}">

File: ulite6_arm_description/urdf/xarm_device_macro.xacro (robot description, xacro)
@@ -1,5 +1,5 @@
 <?xml version='1.0' encoding='utf-8'?>
-<robot xmlns:xacro="http://ros.org/wiki/xacro" name="xarm_device">
-  <xacro:macro name="xarm_device" params="
+<robot xmlns:xacro="http://ros.org/wiki/xacro" name="lite6_device">
+  <xacro:macro name="lite6_device" params="
     prefix:=''
     hw_ns:='xarm'
@@ -9,7 +9,4 @@
     add_gripper:=false
     add_vacuum_gripper:=false
-    add_bio_gripper:=false
-    dof:=7
-    robot_type:='xarm'
     ros2_control_plugin:='uf_robot_hardware/UFRobotSystemHardware'
     attach_to:='world'
@@ -38,5 +35,4 @@
     baud_checkset:=true
     default_gripper_baud:=2000000
-    model1300:=false
     robot_sn:=''
     mesh_suffix:='stl'
@@ -46,8 +42,8 @@
     >
     <!-- Load Common Material -->
-    <xacro:include filename="$(find xarm_description)/urdf/_private_macro.xacro" />
+    <xacro:include filename="$(find ulite6_arm_description)/urdf/private_macro.xacro" />
     <xacro:device_macro_begin />
     <!-- Load Common Material -->
-    <xacro:include filename="$(find xarm_description)/urdf/common/common.material.xacro" />
+    <xacro:include filename="$(find ulite6_arm_description)/urdf/common/common.material.xacro" />
     <xacro:common_material prefix="${prefix}"/>
     <!-- Specify Mesh file path -->
@@ -55,15 +51,15 @@
     <xacro:if value="${ros2_control_plugin == 'gazebo_ros2_control/GazeboSystem' or ros2_control_plugin == 'ign_ros2_control/IgnitionSystem' or ros2_control_plugin == 'gz_ros2_control/GazeboSimSystem'}">
       <!-- gazebo use -->
-      <xacro:property name="mesh_path" value="file://$(find xarm_description)/meshes" scope="parent"/>
+      <xacro:property name="mesh_path" value="file://$(find ulite6_arm_description)/meshes" scope="parent"/>
     </xacro:if>
     <xacro:unless value="${ros2_control_plugin == 'gazebo_ros2_control/GazeboSystem' or ros2_control_plugin == 'ign_ros2_control/IgnitionSystem' or ros2_control_plugin == 'gz_ros2_control/GazeboSimSystem'}">
-      <xacro:property name="mesh_path" value="package://xarm_description/meshes" scope="parent"/>
+      <xacro:property name="mesh_path" value="package://ulite6_arm_description/meshes" scope="parent"/>
     </xacro:unless>
     <!-- include common.link.xacro -->
-    <xacro:include filename="$(find xarm_description)/urdf/common/common.link.xacro" />
-    <xacro:parse_link_inertial_filename dof="${dof}" robot_type="${robot_type}" robot_sn="${robot_sn}" model1300="${model1300}" />
+    <xacro:include filename="$(find ulite6_arm_description)/urdf/common/common.link.xacro" />
+    <xacro:parse_link_inertial_filename dof="6" robot_type="lite" robot_sn="${robot_sn}" model1300="false" />
     <xacro:property name="inertial_params_filename" value="${scope_parent_inertial_params_filename}"/>
     <xacro:property name="model_num" value="${scope_parent_model_num}"/>
-    <!-- add one world link if no 'attach_to' specified  -->
+    <!-- add one world link if no 'attach_to' specified -->
     <xacro:if value="${attach_to == 'world' and create_attach_link}">
       <link name="world" />
@@ -85,127 +81,31 @@
       </xacro:unless>
     </xacro:unless>
-    <xacro:if value="${robot_type == 'uf850' or robot_type == 'xarm7_mirror'}">
-      <xacro:property name="robot_name" value="${robot_type}" />
-    </xacro:if>
-    <xacro:unless value="${robot_type == 'uf850' or robot_type == 'xarm7_mirror'}">
-      <xacro:property name="robot_name" value="${robot_type}${dof}" />
-    </xacro:unless>
+    <xacro:property name="robot_name" value="lite6" />
     <xacro:if value="${kinematics_suffix != ''}">
-      <xacro:property name="kinematics_params_filename" value="$(find xarm_description)/config/kinematics/user/${robot_name}_kinematics_${kinematics_suffix}.yaml"/>
+      <xacro:property name="kinematics_params_filename" value="$(find ulite6_arm_description)/config/kinematics/user/${robot_name}_kinematics_${kinematics_suffix}.yaml"/>
     </xacro:if>
     <xacro:unless value="${kinematics_suffix != ''}">
-      <xacro:property name="kinematics_params_filename" value="$(find xarm_description)/config/kinematics/default/${robot_name}_default_kinematics.yaml"/>
+      <xacro:property name="kinematics_params_filename" value="$(find ulite6_arm_description)/config/kinematics/default/${robot_name}_default_kinematics.yaml"/>
     </xacro:unless>
-    <xacro:if value="${dof == 5}">
-      <!-- Load XArm5 Robot Model URDF -->
-      <xacro:include filename="$(find xarm_description)/urdf/xarm5/xarm5_robot_macro.xacro" />
-      <xacro:xarm5_robot prefix="${prefix}" hw_ns="${hw_ns}" limited="${limited}"
-        velocity_control="${velocity_control}"
-        ros2_control_plugin="${ros2_control_plugin}"
-        add_gripper="${add_gripper}"
-        add_bio_gripper="${add_bio_gripper}"
-        robot_ip="${robot_ip}"
-        report_type="${report_type}"
-        baud_checkset="${baud_checkset}"
-        default_gripper_baud="${default_gripper_baud}"
-        model_num="${model_num}"
-        inertial_params_filename="${inertial_params_filename}"
-        kinematics_params_filename="${kinematics_params_filename}"
-        hard_interface="${hard_interface}" />
-    </xacro:if>
-    <xacro:if value="${dof == 6}">
-      <xacro:if value="${robot_type == 'uf850'}">
-        <!-- Load UFACTORY 850 Robot Model URDF -->
-        <xacro:include filename="$(find xarm_description)/urdf/uf850/uf850_robot_macro.xacro" />
-        <xacro:uf850_robot prefix="${prefix}" hw_ns="${hw_ns}" limited="${limited}"
-          velocity_control="${velocity_control}"
-          ros2_control_plugin="${ros2_control_plugin}"
-          add_gripper="${add_gripper}"
-          add_bio_gripper="${add_bio_gripper}"
-          robot_ip="${robot_ip}"
-          report_type="${report_type}"
-          baud_checkset="${baud_checkset}"
-          default_gripper_baud="${default_gripper_baud}"
-          model_num="${model_num}"
-          inertial_params_filename="${inertial_params_filename}"
-          kinematics_params_filename="${kinematics_params_filename}"
-          hard_interface="${hard_interface}" />
-      </xacro:if>
-      <xacro:if value="${robot_type == 'lite'}">
-        <!-- Load Lite6 Robot Model URDF -->
-        <xacro:include filename="$(find xarm_description)/urdf/lite6/lite6_robot_macro.xacro" />
-        <xacro:lite6_robot prefix="${prefix}" hw_ns="${hw_ns}" limited="${limited}"
-          velocity_control="${velocity_control}"
-          ros2_control_plugin="${ros2_control_plugin}"
-          add_gripper="${add_gripper}"
-          robot_ip="${robot_ip}"
-          report_type="${report_type}"
-          baud_checkset="${baud_checkset}"
-          default_gripper_baud="${default_gripper_baud}"
-          model_num="${model_num}"
-          inertial_params_filename="${inertial_params_filename}"
-          kinematics_params_filename="${kinematics_params_filename}"
-          hard_interface="${hard_interface}" />
-      </xacro:if>
-      <xacro:unless value="${robot_type == 'lite' or robot_type == 'uf850'}">
-        <!-- Load XArm6 Robot Model URDF -->
-        <xacro:include filename="$(find xarm_description)/urdf/xarm6/xarm6_robot_macro.xacro" />
-        <xacro:xarm6_robot prefix="${prefix}" hw_ns="${hw_ns}" limited="${limited}"
-          velocity_control="${velocity_control}"
-          ros2_control_plugin="${ros2_control_plugin}"
-          add_gripper="${add_gripper}"
-          add_bio_gripper="${add_bio_gripper}"
-          robot_ip="${robot_ip}"
-          report_type="${report_type}"
-          baud_checkset="${baud_checkset}"
-          default_gripper_baud="${default_gripper_baud}"
-          model_num="${model_num}"
-          inertial_params_filename="${inertial_params_filename}"
-          kinematics_params_filename="${kinematics_params_filename}"
-          hard_interface="${hard_interface}" />
-      </xacro:unless>
-    </xacro:if>
-    <xacro:unless value="${dof == 5 or dof == 6}">
-      <xacro:if value="${robot_type == 'xarm7_mirror'}">
-        <!-- Load xArm7 Mirror Robot Model URDF -->
-        <xacro:include filename="$(find xarm_description)/urdf/xarm7_mirror/xarm7_mirror_robot_macro.xacro" />
-        <xacro:xarm7_mirror_robot prefix="${prefix}" hw_ns="${hw_ns}" limited="${limited}"
-          velocity_control="${velocity_control}"
-          ros2_control_plugin="${ros2_control_plugin}"
-          add_gripper="${add_gripper}"
-          add_bio_gripper="${add_bio_gripper}"
-          robot_ip="${robot_ip}"
-          report_type="${report_type}"
-          baud_checkset="${baud_checkset}"
-          default_gripper_baud="${default_gripper_baud}"
-          model_num="${model_num}"
-          inertial_params_filename="${inertial_params_filename}"
-          kinematics_params_filename="${kinematics_params_filename}"
-          hard_interface="${hard_interface}" />
-      </xacro:if>
-      <xacro:unless value="${robot_type == 'xarm7_mirror'}">
-        <!-- Load XArm7 Robot Model URDF -->
-        <xacro:include filename="$(find xarm_description)/urdf/xarm7/xarm7_robot_macro.xacro" />
-        <xacro:xarm7_robot prefix="${prefix}" hw_ns="${hw_ns}" limited="${limited}"
-          velocity_control="${velocity_control}"
-          ros2_control_plugin="${ros2_control_plugin}"
-          add_gripper="${add_gripper}"
-          add_bio_gripper="${add_bio_gripper}"
-          robot_ip="${robot_ip}"
-          report_type="${report_type}"
-          baud_checkset="${baud_checkset}"
-          default_gripper_baud="${default_gripper_baud}"
-          model_num="${model_num}"
-          inertial_params_filename="${inertial_params_filename}"
-          kinematics_params_filename="${kinematics_params_filename}"
-          hard_interface="${hard_interface}" />
-      </xacro:unless>
-    </xacro:unless>
+    <!-- Load Lite6 Robot Model URDF -->
+    <xacro:include filename="$(find ulite6_arm_description)/urdf/mech/ulite6_robot_macro.xacro" />
+    <xacro:lite6_robot prefix="${prefix}" hw_ns="${hw_ns}" limited="${limited}"
+      velocity_control="${velocity_control}"
+      ros2_control_plugin="${ros2_control_plugin}"
+      add_gripper="${add_gripper}"
+      robot_ip="${robot_ip}"
+      report_type="${report_type}"
+      baud_checkset="${baud_checkset}"
+      default_gripper_baud="${default_gripper_baud}"
+      model_num="${model_num}"
+      inertial_params_filename="${inertial_params_filename}"
+      kinematics_params_filename="${kinematics_params_filename}"
+      hard_interface="${hard_interface}" />
     <xacro:if value="${add_realsense_d435i}">
       <!-- (xarm) Load RealSense D435i URDF -->
-      <xacro:include filename="$(find xarm_description)/urdf/camera/realsense_d435i.urdf.xacro" />
+      <xacro:include filename="$(find ulite6_arm_description)/urdf/camera/realsense_d435i.urdf.xacro" />
       <xacro:d435i_urdf prefix="${prefix}" add_d435i_links="${add_d435i_links}" />
       <xacro:if value="${add_d435i_links}">
-        <xacro:include filename="$(find xarm_description)/urdf/camera/realsense.gazebo.xacro" />
+        <xacro:include filename="$(find ulite6_arm_description)/urdf/camera/realsense.gazebo.xacro" />
         <xacro:if value="${is_ros2}">
           <xacro:if value="${ros2_control_plugin == 'gz_ros2_control/GazeboSimSystem'}">
@@ -229,47 +129,22 @@
     <joint name="${prefix}joint_eef" type="fixed">
       <origin xyz="0 0 0" rpy="0 0 0" />
-      <parent link="${prefix}link${dof}" />
+      <parent link="${prefix}link6" />
       <child link="${prefix}link_eef" />
     </joint>
     <xacro:if value="${add_gripper}">
-      <xacro:if value="${robot_type == 'lite'}">
-        <!-- Load Lite Gripper Model URDF -->
-        <xacro:include filename="$(find xarm_description)/urdf/gripper/uflite_gripper_macro.xacro" />
-        <xacro:uflite_gripper_macro prefix="${prefix}" attach_to="${prefix}link_eef"
-          ros2_control_plugin="${ros2_control_plugin}" dof="${dof}" hard_interface="${hard_interface}"
-          gripper_version="${gripper_version}" />
-      </xacro:if>
-      <xacro:unless value="${robot_type == 'lite'}">
-        <!-- Load XArm Gripper Model URDF -->
-        <xacro:include filename="$(find xarm_description)/urdf/gripper/xarm_gripper_macro.xacro" />
-        <xacro:xarm_gripper_macro prefix="${prefix}" attach_to="${prefix}link_eef"
-          ros2_control_plugin="${ros2_control_plugin}" dof="${dof}" hard_interface="${hard_interface}"
-          gripper_version="${gripper_version}" />
-      </xacro:unless>
+      <!-- Load Lite Gripper Model URDF -->
+      <xacro:include filename="$(find ulite6_arm_description)/urdf/mech/uflite_gripper_macro.xacro" />
+      <xacro:uflite_gripper_macro prefix="${prefix}" attach_to="${prefix}link_eef"
+        ros2_control_plugin="${ros2_control_plugin}" dof="6" hard_interface="${hard_interface}"
+        gripper_version="${gripper_version}" />
     </xacro:if>
-    <xacro:if value="${not add_gripper and add_bio_gripper}">
-      <xacro:unless value="${robot_type == 'lite'}">
-        <!-- Load BIO Gripper Model URDF -->
-        <xacro:include filename="$(find xarm_description)/urdf/gripper/bio_gripper_macro.xacro" />
-        <xacro:bio_gripper_macro prefix="${prefix}" attach_to="${prefix}link_eef"
-          ros2_control_plugin="${ros2_control_plugin}" dof="${dof}" hard_interface="${hard_interface}"
-          gripper_version="${gripper_version}" />
-      </xacro:unless>
-    </xacro:if>
-    <xacro:if value="${not add_gripper and not add_bio_gripper and add_vacuum_gripper}">
-      <xacro:if value="${robot_type == 'lite'}">
-        <!-- Load Lite Vacuum Gripper Model URDF -->
-        <xacro:include filename="$(find xarm_description)/urdf/vacuum_gripper/lite_vacuum_gripper.urdf.xacro" />
-        <xacro:uflite_vacuum_gripper_urdf prefix="${prefix}" attach_to="${prefix}link_eef" />
-      </xacro:if>
-      <xacro:unless value="${robot_type == 'lite'}">
-        <!-- Load XArm Vacuum Gripper Model URDF -->
-        <xacro:include filename="$(find xarm_description)/urdf/vacuum_gripper/xarm_vacuum_gripper.urdf.xacro" />
-        <xacro:xarm_vacuum_gripper_urdf prefix="${prefix}" attach_to="${prefix}link_eef" />
-      </xacro:unless>
+    <xacro:if value="${not add_gripper and add_vacuum_gripper}">
+      <!-- Load Lite Vacuum Gripper Model URDF -->
+      <xacro:include filename="$(find ulite6_arm_description)/urdf/mech/lite_vacuum_gripper.urdf.xacro" />
+      <xacro:uflite_vacuum_gripper_urdf prefix="${prefix}" attach_to="${prefix}link_eef" />
     </xacro:if>
     <xacro:if value="${not add_gripper and not add_vacuum_gripper and add_other_geometry}">
       <!-- Load Other Model URDF -->
-      <xacro:include filename="$(find xarm_description)/urdf/other/other_geometry.urdf.xacro" />
+      <xacro:include filename="$(find ulite6_arm_description)/urdf/other/other_geometry.urdf.xacro" />
       <xacro:other_geometry prefix="${prefix}" attach_to="${prefix}link_eef"
         geometry_type="${geometry_type}" geometry_mass="${geometry_mass}"
@@ -283,12 +158,7 @@
     <!-- gazebo_plugin -->
     <xacro:if value="${load_gazebo_plugin}">
-      <xacro:include filename="$(find xarm_description)/urdf/common/common.gazebo.xacro" />
+      <xacro:include filename="$(find ulite6_arm_description)/urdf/common/common.gazebo.xacro" />
       <xacro:if value="${is_ros2}">
-        <xacro:if value="${robot_type == 'uf850' or robot_type == 'xarm7_mirror'}">
-          <xacro:property name="new_ros2_control_params" value="$(find xarm_controller)/config/${robot_type}_controllers.yaml"/>
-        </xacro:if>
-        <xacro:unless value="${robot_type == 'uf850' or robot_type == 'xarm7_mirror'}">
-          <xacro:property name="new_ros2_control_params" value="$(find xarm_controller)/config/${robot_type}${dof}_controllers.yaml"/>
-        </xacro:unless>
+        <xacro:property name="new_ros2_control_params" value="$(find xarm_controller)/config/lite6_controllers.yaml"/>
         <xacro:if value="${ros2_control_params != ''}">
           <xacro:property name="new_ros2_control_params" value="${ros2_control_params}"/>
@@ -309,5 +179,5 @@
     </xacro:if>
     <xacro:if value="${use_gazebo_camera}">
-      <xacro:include filename="$(find xarm_description)/urdf/camera/camera.gazebo.xacro" />
+      <xacro:include filename="$(find ulite6_arm_description)/urdf/camera/camera.gazebo.xacro" />
       <xacro:camera_gazebo prefix="${prefix}" />
     </xacro:if>
