Commit message: Cambio en las rutas de las carpetas para poder ejecutar el archivo ulite6_rviz_display.launch.py

File: ulite6_arm_description/urdf/mech/uflite_gripper_macro.xacro (robot description, xacro)
@@ -2,8 +2,8 @@
 <robot xmlns:xacro="http://ros.org/wiki/xacro" name="xarm_gripper" >
   <!-- xarm_gripper -->
-  <xacro:include filename="$(find ulite6_arm_description)/urdf/gripper/uflite_gripper.ros2_control.xacro" />
-  <xacro:include filename="$(find ulite6_arm_description)/urdf/gripper/uflite_gripper.urdf.xacro" />
-  <xacro:include filename="$(find ulite6_arm_description)/urdf/gripper/uflite_gripper.transmission.xacro" />
-  <xacro:include filename="$(find ulite6_arm_description)/urdf/gripper/uflite_gripper.gazebo.xacro" />
+  <xacro:include filename="$(find ulite6_arm_description)/urdf/mech/uflite_gripper.ros2_control.xacro" />
+  <xacro:include filename="$(find ulite6_arm_description)/urdf/mech/gripper.urdf.xacro" />
+  <xacro:include filename="$(find ulite6_arm_description)/urdf/mech/uflite_gripper.transmission.xacro" />
+  <xacro:include filename="$(find ulite6_arm_description)/urdf/mech/uflite_gripper.gazebo.xacro" />
   <xacro:macro name="uflite_gripper_macro" params="prefix:='' attach_to:='' ns:='xarm' attach_xyz:='0 0 0' attach_rpy:='0 0 0'
     ros2_control_plugin:='uf_robot_hardware/UFRobotFakeSystemHardware' dof:=7 hard_interface:='PositionJointInterface' gripper_version:='G1'">

File: ulite6_arm_description/urdf/mech/ulite6_robot_macro.xacro (robot description, xacro)
@@ -21,5 +21,5 @@
       <xacro:include filename="$(find ulite6_arm_description)/urdf/mech/ulite6.ros2_control.xacro" />
     </xacro:if>
-    <xacro:include filename="$(find ulite6_arm_description)/urdf/mech/ulite6.urdf.xacro" />
+    <xacro:include filename="$(find ulite6_arm_description)/urdf/mech/ulite6_arm.urdf.xacro" />
     <xacro:include filename="$(find ulite6_arm_description)/urdf/mech/ulite6.transmission.xacro" />
     <xacro:include filename="$(find ulite6_arm_description)/urdf/mech/ulite6.gazebo.xacro" />

File: ulite6_arm_description/urdf/ulite6_device.urdf.xacro (robot description, xacro)
@@ -8,9 +8,5 @@
   <xacro:arg name="add_gripper" default="false"/>
   <xacro:arg name="add_vacuum_gripper" default="false"/>
-  <xacro:arg name="add_bio_gripper" default="false"/>
-  <xacro:arg name="model1300" default="false"/>
-  <xacro:arg name="dof" default="7"/>
   <xacro:arg name="robot_ip" default=""/>
-  <xacro:arg name="robot_type" default="xarm"/>
   <xacro:arg name="robot_sn" default=""/>
   <xacro:arg name="report_type" default="normal"/>
@@ -40,11 +36,10 @@
   <xacro:arg name="kinematics_suffix" default=""/>
   <xacro:arg name="gripper_version" default="G1"/>
-  <!-- load xarm device -->
-  <xacro:include filename="$(find ulite6_arm_description)/urdf/xarm_device_macro.xacro" />
-  <xacro:xarm_device prefix="$(arg prefix)" hw_ns="$(arg hw_ns)" limited="$(arg limited)"
+  <!-- load ulite6 device -->
+  <xacro:include filename="$(find ulite6_arm_description)/urdf/ulite6_device_macro.xacro" />
+  <xacro:ulite6_device prefix="$(arg prefix)" hw_ns="$(arg hw_ns)" limited="$(arg limited)"
     effort_control="$(arg effort_control)" velocity_control="$(arg velocity_control)"
     add_gripper="$(arg add_gripper)" add_vacuum_gripper="$(arg add_vacuum_gripper)"
-    add_bio_gripper="$(arg add_bio_gripper)" dof="$(arg dof)"
-    ros2_control_plugin="$(arg ros2_control_plugin)" robot_type="$(arg robot_type)"
+    ros2_control_plugin="$(arg ros2_control_plugin)"
     load_gazebo_plugin="true" ros2_control_params="$(arg ros2_control_params)"
     add_realsense_d435i="$(arg add_realsense_d435i)"
@@ -59,5 +54,5 @@
     robot_ip="$(arg robot_ip)" report_type="$(arg report_type)"
     baud_checkset="$(arg baud_checkset)" default_gripper_baud="$(arg default_gripper_baud)"
-    model1300="$(arg model1300)" attach_to="$(arg attach_to)" attach_xyz="$(arg attach_xyz)" attach_rpy="$(arg attach_rpy)"
+    attach_to="$(arg attach_to)" attach_xyz="$(arg attach_xyz)" attach_rpy="$(arg attach_rpy)"
     robot_sn="$(arg robot_sn)" use_gazebo_camera="$(arg use_gazebo_camera)" mesh_suffix="$(arg mesh_suffix)" kinematics_suffix="$(arg kinematics_suffix)"
     gripper_version="$(arg gripper_version)" />

File: ulite6_arm_description/urdf/ulite6_device_macro.xacro (robot description, xacro)
@@ -1,5 +1,5 @@
 <?xml version='1.0' encoding='utf-8'?>
 <robot xmlns:xacro="http://ros.org/wiki/xacro" name="lite6_device">
-  <xacro:macro name="lite6_device" params="
+  <xacro:macro name="ulite6_device" params="
     prefix:=''
     hw_ns:='xarm'
@@ -141,5 +141,5 @@
     <xacro:if value="${not add_gripper and add_vacuum_gripper}">
       <!-- Load Lite Vacuum Gripper Model URDF -->
-      <xacro:include filename="$(find ulite6_arm_description)/urdf/mech/lite_vacuum_gripper.urdf.xacro" />
+      <xacro:include filename="$(find ulite6_arm_description)/urdf/mech/ulite6_vacuum_gripper.urdf.xacro" />
       <xacro:uflite_vacuum_gripper_urdf prefix="${prefix}" attach_to="${prefix}link_eef" />
     </xacro:if>

Commit message: Se creo el  archivo ulite6_draw_square.launch.py para trazar trayectorias de figuras geométricas básicas sobre el canvas

File: ulite6_arm_description/urdf/mech/uflite_gripper_macro.xacro (robot description, xacro)
@@ -18,7 +18,12 @@
     </xacro:if>
     <!-- mimic_joint_plugin has to be installed: -->
-    <xacro:mimic_joint_plugin_gazebo name_prefix="${prefix}finger_joint2"
-      following_joint="${prefix}finger_joint1" mimic_joint="${prefix}finger_joint2"
-      has_pid="${is_ros2}" multiplier="1.0" max_effort="10.0" />
+    <!-- gz-sim (Gazebo Sim) e Ignition resuelven la etiqueta <mimic> del URDF de
+         forma nativa (motor bullet-featherstone), por lo que este plugin de
+         Gazebo Classic solo se carga con gazebo_ros2_control o ROS 1 -->
+    <xacro:unless value="${ros2_control_plugin == 'gz_ros2_control/GazeboSimSystem' or ros2_control_plugin == 'ign_ros2_control/IgnitionSystem'}">
+      <xacro:mimic_joint_plugin_gazebo name_prefix="${prefix}finger_joint2"
+        following_joint="${prefix}finger_joint1" mimic_joint="${prefix}finger_joint2"
+        has_pid="${is_ros2}" multiplier="1.0" max_effort="10.0" />
+    </xacro:unless>
   </xacro:macro>
 </robot>
